File: pcb/LTC3112_buck-boost.brd (EAGLE design)
At the start: 43.2 x 32.3 mm, 18 parts

Commit message: noty + pcb
Routing:
- net GND: track 41.6 -> 40.6 mm
Changed lines of the file:
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@@
 <wire x1="28.702" y1="11.43" x2="31.242" y2="11.43" width="0.3048" layer="1"/>
 <wire x1="31.242" y1="11.43" x2="31.75" y2="11.938" width="0.6096" layer="1"/>
-<wire x1="31.75" y1="11.938" x2="31.75" y2="12.866" width="0.3048" layer="1" curve="356.335724"/>
 <wire x1="31.75" y1="12.866" x2="31.8253" y2="12.7762" width="0.3048" layer="1"/>
 <wire x1="22.475" y1="16.1322" x2="21.7138" y2="16.1322" width="0.3048" layer="1"/>
