File: pcb/max9611.sch (EAGLE design)
At the start: 14 parts

Commit message: dodanie worda z magisterką gdzie pisze na bierząco, update kosztorysu, nowe bordy
Parts:
- renumbered PAD1 to ANL
Changed lines of the file:
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@@
 <part name="GND5" library="supply1" deviceset="GND" device=""/>
 <part name="P+6" library="supply1" deviceset="VCC" device=""/>
-<part name="PAD1" library="wirepad" deviceset="1,6/0,8" device=""/>
+<part name="ANL" library="wirepad" deviceset="1,6/0,8" device=""/>
 <part name="J4" library="con-amp" deviceset="MTA02-100" device=""/>
 <part name="P+7" library="supply1" deviceset="VCC" device=""/>
@@
 <instance part="GND5" gate="1" x="68.58" y="38.1"/>
 <instance part="P+6" gate="VCC" x="68.58" y="53.34"/>
-<instance part="PAD1" gate="P" x="83.82" y="68.58"/>
+<instance part="ANL" gate="P" x="83.82" y="68.58"/>
 <instance part="J4" gate="G$1" x="86.36" y="91.44"/>
 <instance part="P+7" gate="VCC" x="86.36" y="86.36" rot="R180"/>
@@
 <segment>
 <pinref part="U$1" gate="G$1" pin="OUT"/>
-<pinref part="PAD1" gate="P" pin="P"/>
+<pinref part="ANL" gate="P" pin="P"/>
 </segment>
 </net>
