File: pcb/ogranicznik_napiecia.brd (EAGLE design)
At the start: 27.9 x 25.1 mm, 6 parts, among them T1 BD235

Commit message: fuel gauge tutorial, mgr update
Parts:
- removed PAD2: (no value), wirepad:2,54/0,9
- removed T1: BD235, transistor:TO126
- added Q1: BD139, transistor-power:TO126AV
- added U$2: MAX6129, ref-packages:SOT23-5L
- R1: value (none) -> 100k
- R2: value (none) -> 1k
- renumbered PAD1 to VCCIN
Connections:
- net GND: now also Q1.E, U$2.1; no longer T1.1
- net N$1: now also Q1.B; no longer T1.3
- net N$4: now also U$2.5; no longer PAD2.1
- net VCC: now also Q1.C, U$2.2; no longer T1.2
Routing:
- net GND: track 10.5 -> 23.4 mm, vias 0 -> 2
- net VCC: track 64.3 -> 66.0 mm

Commit message: rewizja bordów
Parts:
- added C1, C2: 10u/6,3v, rcl:SMC_B
- added C3, C4: 100n, rcl:C0805
- moved U$2 2.83 mm to (11.1, 17.9)
- moved VCCIN 1.27 mm to (3.81, 3.81)
Connections:
- net GND: now also C1.-, C2.-, C3.2, C4.2, U$2.2; no longer U$2.1
- net N$4: now also C1.+
- net VCC: now also C2.+, C3.1, C4.1, U$2.1; no longer U$2.2
Routing:
- net VCC: track 66.0 -> 70.0 mm
- net GND: track 23.4 -> 27.3 mm
- net N$4: track 6.87 -> 9.11 mm
Other:
- board size 27.9 x 25.1 mm -> 24.9 x 24.6 mm
Changed lines of the file:
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@@
 <board>
 <plain>
-<wire x1="0" y1="0" x2="27.92" y2="0" width="0" layer="20"/>
-<wire x1="27.92" y1="0" x2="27.92" y2="25.07" width="0" layer="20"/>
-<wire x1="27.92" y1="25.07" x2="0" y2="25.07" width="0" layer="20"/>
-<wire x1="0" y1="25.07" x2="0" y2="0" width="0" layer="20"/>
+<wire x1="1.39519375" y1="0.865796875" x2="26.2178625" y2="0.80994375" width="0" layer="20"/>
+<wire x1="26.2178625" y1="0.80994375" x2="26.162053125" y2="25.40515" width="0" layer="20"/>
+<wire x1="26.162053125" y1="25.40515" x2="1.31148125" y2="25.377215625" width="0" layer="20"/>
+<wire x1="1.31148125" y1="25.377215625" x2="1.39519375" y2="0.865796875" width="0" layer="20"/>
 </plain>
 <attributes>
@@
 <classes>
 <class number="0" name="default" width="0" drill="0">
-<clearance class="0" value="0.65"/>
+<clearance class="0" value="0.75"/>
 </class>
 </classes>
@@
 <element name="R1" library="pot" package="RJ9W" value="100k" x="5.08" y="13.97" rot="R270"/>
 <element name="R2" library="rcl" package="M0805" value="1k" x="19.05" y="6.35" rot="R180"/>
-<element name="VCCIN" library="wirepad" package="2,54/0,9" value="" x="5.08" y="3.81"/>
-<element name="U$2" library="ref-packages" package="SOT23-5L" value="MAX6129" x="13.8623375" y="18.552009375" rot="R180"/>
+<element name="VCCIN" library="wirepad" package="2,54/0,9" value="" x="3.81" y="3.81"/>
+<element name="U$2" library="ref-packages" package="SOT23-5L" value="MAX6129" x="11.1178" y="17.8523875" rot="R180"/>
 <element name="Q1" library="transistor-power" package="TO126AV" value="BD139" x="12.7" y="7.62"/>
+<element name="C1" library="rcl" package="SMC_B" value="10u/6,3v" x="16.112515625" y="16.922425"/>
+<element name="C2" library="rcl" package="SMC_B" value="10u/6,3v" x="7.0579375" y="5.390046875" rot="R90"/>
+<element name="C3" library="rcl" package="C0805" value="100n" x="20.4431125" y="14.427771875" rot="R90"/>
+<element name="C4" library="rcl" package="C0805" value="100n" x="12.0365875" y="22.64595625" rot="R90"/>
 </elements>
 <signals>
@@
 <vertex x="-5.08" y="31.75"/>
 </polygon>
-<contactref element="U$2" pad="1"/>
+<contactref element="U$2" pad="2"/>
 <contactref element="Q1" pad="E"/>
 <wire x1="10.414" y1="6.35" x2="7.62" y2="9.144" width="0.8128" layer="1"/>
 <wire x1="7.62" y1="9.144" x2="7.62" y2="10.795" width="0.8128" layer="1"/>
-<wire x1="14.8123375" y1="19.852009375" x2="15.759378125" y2="18.90496875" width="0.6096" layer="1"/>
-<wire x1="15.759378125" y1="18.90496875" x2="18.940246875" y2="18.90496875" width="0.6096" layer="1"/>
-<via x="18.940246875" y="18.90496875" extent="1-16" drill="0.6"/>
-<wire x1="18.940246875" y1="18.90496875" x2="22.71496875" y2="18.90496875" width="0.6096" layer="16"/>
-<wire x1="22.71496875" y1="18.90496875" x2="24.13" y2="20.32" width="0.6096" layer="16"/>
-<via x="24.13" y="20.32" extent="1-16" drill="0.6"/>
-<wire x1="24.13" y1="20.32" x2="24.13" y2="21.59" width="0.6096" layer="1"/>
+<contactref element="C2" pad="-"/>
+<contactref element="C1" pad="-"/>
+<contactref element="C3" pad="2"/>
+<contactref element="C4" pad="2"/>
+<wire x1="16.743278125" y1="19.596378125" x2="20.0862125" y2="17.79995" width="0.6096" layer="1"/>
+<via x="20.0862125" y="17.79995" extent="1-16" drill="0.8" diameter="1.9304"/>
+<wire x1="20.0862125" y1="17.79995" x2="21.9561875" y2="19.777721875" width="0.6096" layer="16"/>
+<wire x1="21.9561875" y1="19.777721875" x2="23.570696875" y2="21.39223125" width="0.6096" layer="16"/>
+<via x="23.570696875" y="21.39223125" extent="1-16" drill="0.8" diameter="1.9304"/>
+<wire x1="23.570696875" y1="21.39223125" x2="23.570696875" y2="22.300696875" width="0.6096" layer="1"/>
+<wire x1="23.570696875" y1="22.300696875" x2="24.13" y2="22.86" width="0.6096" layer="1"/>
+<wire x1="11.1178" y1="19.1523875" x2="11.1178" y2="18.00739375" width="0.6096" layer="1"/>
+<wire x1="11.1178" y1="18.00739375" x2="11.330603125" y2="17.794590625" width="0.6096" layer="1"/>
+<wire x1="11.330603125" y1="17.794590625" x2="12.563609375" y2="17.794590625" width="0.6096" layer="1"/>
+<wire x1="12.563609375" y1="17.794590625" x2="12.89054375" y2="18.121525" width="0.6096" layer="1"/>
+<wire x1="12.89054375" y1="18.121525" x2="12.89054375" y2="18.915509375" width="0.6096" layer="1"/>
+<wire x1="12.89054375" y1="18.915509375" x2="13.553753125" y2="19.57871875" width="0.6096" layer="1"/>
 </signal>
 <signal name="N$1">
@@
 <contactref element="U$1" pad="7"/>
 <contactref element="VCCIN" pad="1"/>
-<wire x1="5.715" y1="16.51" x2="5.715" y2="18.415" width="0.8128" layer="1"/>
-<wire x1="5.715" y1="18.415" x2="8.89" y2="21.59" width="0.8128" layer="1"/>
-<wire x1="8.89" y1="21.59" x2="13.875028125" y2="21.59" width="0.8128" layer="1"/>
-<wire x1="13.875028125" y1="21.59" x2="20.32" y2="21.59" width="0.8128" layer="1"/>
-<wire x1="20.32" y1="21.59" x2="22.86" y2="17.78" width="0.8128" layer="1"/>
+<wire x1="5.715" y1="16.51" x2="5.715" y2="18.415" width="1.016" layer="1"/>
+<wire x1="5.715" y1="18.415" x2="8.89" y2="21.59" width="1.016" layer="1"/>
+<wire x1="8.89" y1="21.59" x2="11.184309375" y2="21.670725" width="1.016" layer="1"/>
+<wire x1="11.184309375" y1="21.670725" x2="12.0703625" y2="21.6692875" width="1.016" layer="1"/>
+<wire x1="12.0703625" y1="21.6692875" x2="20.346909375" y2="21.657271875" width="1.016" layer="1"/>
+<wire x1="20.346909375" y1="21.657271875" x2="22.86" y2="17.78" width="1.016" layer="1"/>
 <wire x1="16.57" y1="13.335" x2="22.225" y2="13.335" width="0.6096" layer="1"/>
 <wire x1="22.225" y1="13.335" x2="22.86" y2="13.97" width="0.6096" layer="1"/>
-<wire x1="22.86" y1="13.97" x2="22.86" y2="17.78" width="0.8128" layer="1"/>
-<wire x1="5.08" y1="3.81" x2="12.7" y2="3.81" width="0.8128" layer="1"/>
-<wire x1="12.7" y1="3.81" x2="13.97" y2="2.54" width="0.8128" layer="1"/>
-<wire x1="13.97" y1="2.54" x2="21.59" y2="2.54" width="0.8128" layer="1"/>
-<wire x1="21.59" y1="2.54" x2="22.86" y2="3.81" width="0.8128" layer="1"/>
-<wire x1="22.86" y1="3.81" x2="22.86" y2="13.97" width="0.8128" layer="1"/>
-<contactref element="U$2" pad="2"/>
+<wire x1="22.86" y1="13.97" x2="22.86" y2="17.78" width="1.016" layer="1"/>
+<wire x1="3.81" y1="3.81" x2="12.7" y2="3.81" width="1.016" layer="1"/>
+<wire x1="12.7" y1="3.81" x2="13.97" y2="2.54" width="1.016" layer="1"/>
+<wire x1="13.97" y1="2.54" x2="21.59" y2="2.54" width="1.016" layer="1"/>
+<wire x1="21.59" y1="2.54" x2="22.86" y2="3.81" width="1.016" layer="1"/>
+<wire x1="22.86" y1="3.81" x2="22.86" y2="13.97" width="1.016" layer="1"/>
+<contactref element="U$2" pad="1"/>
 <contactref element="Q1" pad="C"/>
-<wire x1="12.7" y1="6.35" x2="12.7" y2="3.81" width="0.8128" layer="1"/>
-<wire x1="13.8623375" y1="19.852009375" x2="13.875028125" y2="19.8647" width="0.6096" layer="1"/>
-<wire x1="13.875028125" y1="19.8647" x2="13.875028125" y2="21.59" width="0.6096" layer="1"/>
+<wire x1="12.7" y1="6.35" x2="12.7" y2="3.81" width="1.016" layer="1"/>
+<contactref element="C2" pad="+"/>
+<contactref element="C3" pad="1"/>
+<contactref element="C4" pad="1"/>
+<wire x1="22.225" y1="13.335" x2="20.585884375" y2="13.335" width="0.8128" layer="1"/>
+<wire x1="20.585884375" y1="13.335" x2="20.4431125" y2="13.477771875" width="0.8128" layer="1"/>
+<wire x1="12.0678" y1="19.1523875" x2="12.0703625" y2="19.596378125" width="0.6096" layer="1"/>
+<wire x1="12.0703625" y1="19.596378125" x2="12.0703625" y2="21.6692875" width="0.6096" layer="1"/>
+<wire x1="12.0703625" y1="21.6692875" x2="12.0365875" y2="21.69595625" width="0" layer="19" extent="1-1"/>
+<wire x1="7.0579375" y1="3.890046875" x2="3.81" y2="3.81" width="0" layer="19" extent="1-1"/>
 </signal>
 <signal name="N$3">
@@
 <signal name="N$4">
 <contactref element="U$1" pad="2"/>
-<wire x1="11.37" y1="13.335" x2="13.97" y2="13.335" width="0.6096" layer="1"/>
 <contactref element="U$2" pad="5"/>
-<wire x1="13.97" y1="13.335" x2="14.2787625" y2="13.6437625" width="0.6096" layer="1"/>
-<wire x1="14.2787625" y1="13.6437625" x2="14.2787625" y2="15.8011625" width="0.6096" layer="1"/>
-<wire x1="14.2787625" y1="15.8011625" x2="14.8123375" y2="16.3347375" width="0.6096" layer="1"/>
-<wire x1="14.8123375" y1="16.3347375" x2="14.8123375" y2="17.252009375" width="0.6096" layer="1"/>
+<contactref element="C1" pad="+"/>
+<wire x1="12.0678" y1="16.5523875" x2="14.5846125" y2="16.5523875" width="0.8128" layer="1"/>
+<wire x1="14.5846125" y1="16.5523875" x2="14.9614625" y2="16.996378125" width="0.4064" layer="1"/>
+<wire x1="14.9614625" y1="16.996378125" x2="14.612515625" y2="16.922425" width="0.4064" layer="1"/>
+<wire x1="11.37" y1="13.335" x2="13.118846875" y2="13.335" width="0.8128" layer="1"/>
+<wire x1="13.118846875" y1="13.335" x2="14.28861875" y2="14.504771875" width="0.8128" layer="1"/>
+<wire x1="14.28861875" y1="14.504771875" x2="14.28861875" y2="16.44475" width="0.8128" layer="1"/>
+<wire x1="14.28861875" y1="16.44475" x2="14.5846125" y2="16.5523875" width="0.4064" layer="1"/>
 </signal>
 </signals>
