File: pcb/LTC3115 - przetwornica ogniwo.brd (EAGLE design)
At the start: 29.2 x 30.8 mm, 15 parts

Commit message: +mgr
Parts:
- added C8: 220u/25v, rcl:E2,5-6E
- added IN: (no value), wirepad:1,6/0,8
- added R6: 160k, rcl:M0805
- C1, C2: value (none) -> 68n
- C3: value (none) -> 4u7/50v
- C4: value (none) -> 330u/10v
- C5: value (none) -> 33n
- C6: value (none) -> 100n
- C7: value (none) -> 47n
- L1: value (none) -> DE0704-10 (10uH)
- R1: value (none) -> 560k; device pot:RJ9W -> rcl:M0805
- R2: value (none) -> 28k
- R3: value (none) -> 33k
- R4: value (none) -> 27k
- R5: value (none) -> 10k
- moved R1 1.14 mm to (17.5, 29.5), turned to 90 degrees
Connections:
- net GND: now also C8.-, R6.1; no longer R1.A
- net N$6: now also R1.1, R6.2; no longer R1.S
- net N$7: now also R1.2; no longer R1.E
- net VDD: now also C8.+, IN.1
Routing:
- net GND: track 8.21 -> 17.2 mm
- net VDD: track 23.1 -> 29.1 mm
- net N$6: track 10.1 -> 13.8 mm
- net N$7: track 18.6 -> 20.6 mm
Other:
- board size 29.2 x 30.8 mm -> 29.5 x 30.8 mm
- board text removed: "SMPS"
