File: pcb/LTC3115 - przetwornica ogniwo.sch (EAGLE design)
At the start: 15 parts

Commit message: +mgr
Parts:
- added C8: 220u/25v, rcl:CPOL-EUE2,5-6E
- added IN: (no value), wirepad:1,6/0,8
- added R6: 160k, rcl:R-EU_M0805
- C1, C2: value (none) -> 68n
- C3: value (none) -> 4u7/50v
- C4: value (none) -> 330u/10v
- C5: value (none) -> 33n
- C6: value (none) -> 100n
- C7: value (none) -> 47n
- L1: value (none) -> DE0704-10 (10uH)
- R1: value (none) -> 560k; device pot:TRIM_EU-RJ9W -> rcl:R-EU_M0805
- R2: value (none) -> 28k
- R3: value (none) -> 33k
- R4: value (none) -> 27k
- R5: value (none) -> 10k
Connections:
- net GND: now also C8.-, R6.1; no longer R1.A
- net N$6: now also R1.1, R6.2; no longer R1.S
- net N$7: now also R1.2; no longer R1.E
- net VDD: now also C8.+, IN.P
Other:
- moved on the sheet: C2
Changed lines of the file:
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@@
 <parts>
 <part name="U$1" library="ref-packages" deviceset="LTC3114" device=""/>
-<part name="C1" library="resistor" deviceset="C-EU" device="C0805"/>
-<part name="C2" library="resistor" deviceset="C-EU" device="C0805"/>
-<part name="L1" library="rcl" deviceset="L-EU" device="L3225M"/>
+<part name="C1" library="resistor" deviceset="C-EU" device="C0805" value="68n"/>
+<part name="C2" library="resistor" deviceset="C-EU" device="C0805" value="68n"/>
+<part name="L1" library="rcl" deviceset="L-EU" device="L3225M" value="DE0704-10 (10uH)"/>
 <part name="VDD1" library="supply1" deviceset="VDD" device=""/>
 <part name="VDD2" library="supply1" deviceset="VDD" device=""/>
-<part name="C3" library="rcl" deviceset="CPOL-EU" device="E2,5-6E"/>
+<part name="C3" library="rcl" deviceset="CPOL-EU" device="E2,5-6E" value="4u7/50v"/>
 <part name="GND1" library="supply1" deviceset="GND" device=""/>
 <part name="GND2" library="supply1" deviceset="GND" device=""/>
 <part name="GND3" library="supply1" deviceset="GND" device=""/>
-<part name="R1" library="pot" deviceset="TRIM_EU-" device="RJ9W"/>
 <part name="GND4" library="supply1" deviceset="GND" device=""/>
-<part name="C4" library="rcl" deviceset="CPOL-EU" device="E2,5-6E"/>
+<part name="C4" library="rcl" deviceset="CPOL-EU" device="E2,5-6E" value="330u/10v"/>
 <part name="GND5" library="supply1" deviceset="GND" device=""/>
-<part name="R2" library="rcl" deviceset="R-EU_" device="M0805"/>
-<part name="C5" library="rcl" deviceset="C-EU" device="C0805"/>
+<part name="R2" library="rcl" deviceset="R-EU_" device="M0805" value="28k"/>
+<part name="C5" library="rcl" deviceset="C-EU" device="C0805" value="33n"/>
 <part name="GND6" library="supply1" deviceset="GND" device=""/>
 <part name="OUT" library="wirepad" deviceset="1,6/0,8" device=""/>
-<part name="C7" library="rcl" deviceset="C-EU" device="C0805"/>
-<part name="R4" library="rcl" deviceset="R-EU_" device="M0805"/>
+<part name="C7" library="rcl" deviceset="C-EU" device="C0805" value="47n"/>
+<part name="R4" library="rcl" deviceset="R-EU_" device="M0805" value="27k"/>
 <part name="GND7" library="supply1" deviceset="GND" device=""/>
 <part name="GND8" library="supply1" deviceset="GND" device=""/>
-<part name="R5" library="rcl" deviceset="R-EU_" device="M0805"/>
+<part name="R5" library="rcl" deviceset="R-EU_" device="M0805" value="10k"/>
 <part name="GND9" library="supply1" deviceset="GND" device=""/>
 <part name="VDD3" library="supply1" deviceset="VDD" device=""/>
-<part name="C6" library="rcl" deviceset="C-EU" device="C0805"/>
+<part name="C6" library="rcl" deviceset="C-EU" device="C0805" value="100n"/>
 <part name="GND10" library="supply1" deviceset="GND" device=""/>
-<part name="R3" library="rcl" deviceset="R-EU_" device="M0805"/>
+<part name="R3" library="rcl" deviceset="R-EU_" device="M0805" value="33k"/>
+<part name="R1" library="rcl" deviceset="R-EU_" device="M0805" value="560k"/>
+<part name="R6" library="rcl" deviceset="R-EU_" device="M0805" value="160k"/>
+<part name="C8" library="rcl" deviceset="CPOL-EU" device="E2,5-6E" value="220u/25v"/>
+<part name="VDD4" library="supply1" deviceset="VDD" device=""/>
+<part name="GND11" library="supply1" deviceset="GND" device=""/>
+<part name="IN" library="wirepad" deviceset="1,6/0,8" device=""/>
 </parts>
 <sheets>
@@
 <instance part="U$1" gate="G$1" x="66.04" y="45.72"/>
 <instance part="C1" gate="G$1" x="93.98" y="55.88"/>
-<instance part="C2" gate="G$1" x="68.58" y="88.9" rot="R270"/>
-<instance part="L1" gate="G$1" x="66.04" y="71.12" rot="R90"/>
+<instance part="C2" gate="G$1" x="68.58" y="78.74" smashed="yes" rot="R270">
+<attribute name="NAME" x="66.294" y="82.677" size="1.778" layer="95" rot="R180"/>
+<attribute name="VALUE" x="71.882" y="82.931" size="1.778" layer="96" rot="R180"/>
+</instance>
+<instance part="L1" gate="G$1" x="66.04" y="71.12" smashed="yes" rot="R90">
+<attribute name="NAME" x="69.85" y="69.6214" size="1.778" layer="95" rot="R180"/>
+<attribute name="VALUE" x="80.01" y="74.422" size="1.778" layer="96" rot="R180"/>
+</instance>
 <instance part="VDD1" gate="G$1" x="83.82" y="50.8" rot="R270"/>
 <instance part="VDD2" gate="G$1" x="83.82" y="40.64" rot="R270"/>
@@
 <instance part="GND2" gate="1" x="45.72" y="38.1" rot="R270"/>
 <instance part="GND3" gate="1" x="45.72" y="55.88" rot="R270"/>
-<instance part="R1" gate="1" x="25.4" y="40.64"/>
-<instance part="GND4" gate="1" x="25.4" y="33.02"/>
-<instance part="C4" gate="G$1" x="15.24" y="48.26"/>
+<instance part="GND4" gate="1" x="25.4" y="12.7"/>
+<instance part="C4" gate="G$1" x="15.24" y="48.26" smashed="yes">
+<attribute name="NAME" x="16.383" y="48.7426" size="1.778" layer="95"/>
+<attribute name="VALUE" x="1.905" y="47.2186" size="1.778" layer="96"/>
+</instance>
 <instance part="GND5" gate="1" x="15.24" y="40.64"/>
 <instance part="R2" gate="G$1" x="35.56" y="17.78" rot="R90"/>
@@
 <instance part="GND9" gate="1" x="27.94" y="63.5" rot="R90"/>
 <instance part="VDD3" gate="G$1" x="-2.54" y="63.5" rot="R90"/>
-<instance part="C6" gate="G$1" x="12.7" y="68.58"/>
-<instance part="GND10" gate="1" x="12.7" y="73.66" rot="R180"/>
+<instance part="C6" gate="G$1" x="12.7" y="68.58" smashed="yes">
+<attribute name="NAME" x="14.224" y="68.961" size="1.778" layer="95"/>
+<attribute name="VALUE" x="6.604" y="68.961" size="1.778" layer="96"/>
+</instance>
+<instance part="GND10" gate="1" x="12.7" y="78.74" rot="R180"/>
 <instance part="R3" gate="G$1" x="5.08" y="63.5" rot="R180"/>
+<instance part="R1" gate="G$1" x="25.4" y="40.64" rot="R90"/>
+<instance part="R6" gate="G$1" x="25.4" y="20.32" rot="R90"/>
+<instance part="C8" gate="G$1" x="111.76" y="48.26"/>
+<instance part="VDD4" gate="G$1" x="111.76" y="60.96"/>
+<instance part="GND11" gate="1" x="111.76" y="40.64"/>
+<instance part="IN" gate="P" x="114.3" y="55.88" rot="R180"/>
 </instances>
 <busses>
@@
 <segment>
 <pinref part="U$1" gate="G$1" pin="BST2"/>
-<wire x1="81.28" y1="45.72" x2="104.14" y2="45.72" width="0.1524" layer="91"/>
-<wire x1="104.14" y1="45.72" x2="104.14" y2="88.9" width="0.1524" layer="91"/>
+<wire x1="81.28" y1="45.72" x2="101.6" y2="45.72" width="0.1524" layer="91"/>
+<wire x1="101.6" y1="45.72" x2="101.6" y2="78.74" width="0.1524" layer="91"/>
 <pinref part="C2" gate="G$1" pin="1"/>
-<wire x1="104.14" y1="88.9" x2="71.12" y2="88.9" width="0.1524" layer="91"/>
+<wire x1="101.6" y1="78.74" x2="71.12" y2="78.74" width="0.1524" layer="91"/>
 </segment>
 </net>
@@
 <pinref part="C2" gate="G$1" pin="2"/>
 <wire x1="55.88" y1="71.12" x2="60.96" y2="71.12" width="0.1524" layer="91"/>
-<wire x1="63.5" y1="88.9" x2="55.88" y2="88.9" width="0.1524" layer="91"/>
-<wire x1="55.88" y1="88.9" x2="55.88" y2="71.12" width="0.1524" layer="91"/>
+<wire x1="63.5" y1="78.74" x2="55.88" y2="78.74" width="0.1524" layer="91"/>
+<wire x1="55.88" y1="78.74" x2="55.88" y2="71.12" width="0.1524" layer="91"/>
 <junction x="55.88" y="71.12"/>
 </segment>
@@
 <pinref part="VDD3" gate="G$1" pin="VDD"/>
 <pinref part="R3" gate="G$1" pin="2"/>
+</segment>
+<segment>
+<pinref part="C8" gate="G$1" pin="+"/>
+<pinref part="VDD4" gate="G$1" pin="VDD"/>
+<wire x1="111.76" y1="58.42" x2="111.76" y2="55.88" width="0.1524" layer="91"/>
+<pinref part="IN" gate="P" pin="P"/>
+<wire x1="111.76" y1="55.88" x2="111.76" y2="50.8" width="0.1524" layer="91"/>
+<junction x="111.76" y="55.88"/>
 </segment>
 </net>
@@
 <pinref part="U$1" gate="G$1" pin="PGND"/>
 <pinref part="GND3" gate="1" pin="GND"/>
-</segment>
-<segment>
-<pinref part="R1" gate="1" pin="A"/>
-<pinref part="GND4" gate="1" pin="GND"/>
 </segment>
 <segment>
@@
 <pinref part="C6" gate="G$1" pin="1"/>
 <pinref part="GND10" gate="1" pin="GND"/>
+<wire x1="12.7" y1="76.2" x2="12.7" y2="71.12" width="0.1524" layer="91"/>
+</segment>
+<segment>
+<pinref part="GND4" gate="1" pin="GND"/>
+<pinref part="R6" gate="G$1" pin="1"/>
+</segment>
+<segment>
+<pinref part="C8" gate="G$1" pin="-"/>
+<pinref part="GND11" gate="1" pin="GND"/>
 </segment>
 </net>
@@
 <segment>
 <pinref part="U$1" gate="G$1" pin="FB"/>
-<pinref part="R1" gate="1" pin="S"/>
 <wire x1="48.26" y1="40.64" x2="30.48" y2="40.64" width="0.1524" layer="91"/>
+<wire x1="30.48" y1="40.64" x2="30.48" y2="33.02" width="0.1524" layer="91"/>
+<pinref part="R1" gate="G$1" pin="1"/>
+<pinref part="R6" gate="G$1" pin="2"/>
+<wire x1="25.4" y1="35.56" x2="25.4" y2="33.02" width="0.1524" layer="91"/>
+<wire x1="25.4" y1="33.02" x2="25.4" y2="25.4" width="0.1524" layer="91"/>
+<wire x1="30.48" y1="33.02" x2="25.4" y2="33.02" width="0.1524" layer="91"/>
+<junction x="25.4" y="33.02"/>
 </segment>
 </net>
@@
 <segment>
 <pinref part="U$1" gate="G$1" pin="PVOUT"/>
-<pinref part="R1" gate="1" pin="E"/>
 <wire x1="48.26" y1="50.8" x2="25.4" y2="50.8" width="0.1524" layer="91"/>
 <wire x1="25.4" y1="50.8" x2="25.4" y2="45.72" width="0.1524" layer="91"/>
@@
 <junction x="15.24" y="50.8"/>
 <pinref part="OUT" gate="P" pin="P"/>
-</segment>
-</net>
+<pinref part="R1" gate="G$1" pin="2"/>
+</segment>
+</net>
