File: pcb/GPS_dev_board.sch (EAGLE design)
At the start: 12 parts

Commit message: mgr, pcb uszko
Other:
- moved on the sheet: PAD3
Changed lines of the file:
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@@
 <instance part="PAD1" gate="P" x="25.4" y="50.8"/>
 <instance part="PAD2" gate="P" x="25.4" y="48.26"/>
-<instance part="PAD3" gate="P" x="22.86" y="45.72"/>
+<instance part="PAD3" gate="P" x="25.4" y="45.72"/>
 <instance part="PAD4" gate="P" x="25.4" y="40.64"/>
 <instance part="PAD5" gate="P" x="25.4" y="38.1"/>
@@
 <segment>
 <pinref part="PAD3" gate="P" pin="P"/>
-<wire x1="25.4" y1="45.72" x2="33.02" y2="45.72" width="0.1524" layer="91"/>
+<wire x1="27.94" y1="45.72" x2="33.02" y2="45.72" width="0.1524" layer="91"/>
 <pinref part="U$1" gate="G$1" pin="GND"/>
 </segment>
