File: pcb/bord cyfrowy uszko/uszko.sch (EAGLE design)
At the start: 0 parts

Commit message: bord dla uszka, prezentacja
Parts:
- added BAT+, BAT-, PTE6: (no value), wirepad:2,54/0,8
- added C4: 100n, rcl:C-EUC0805
- added D1, D2: 5V6, diode:ZENER-DIODESOD80C
- added J1, J2: (no value), con-amp:MTA07-100
- added PAD1: (no value), wirepad:2,15/1,0
- added R4: 1k, resistor:R-EU_M0805
- added R5: 500R, resistor:R-EU_M0805
- added R6: 20m, resistor:R-EU_M1206
- added R7, R8: 150R, resistor:R-EU_M0805
- added SL1: (no value), con-amp-quick:M03
- added SL2, SL3: (no value), con-amp-quick:M04
- added U$1: INTO_CON, ref-packages:INTO_CON
- added U$2: GTS-4E-60, ref-packages:GTS-4E-60
- added U$4: SI7020-A10, ref-packages:SI7020-A10
- added U$5: 12PINCON, ref-packages:12PINCON
- added U$6: MAX44006, MAX44006:MAX44006
- added U$7: DS2782, ref-packages:DS2782
- added U1: ADT7410TRZ, ref-packages:ADT7410TRZ
Connections:
- new net +5V/1: J1.6, SL1.1, SL3.4, U$1.3V3, U$2.VCC, U$4.VDD, U$5.P$2, U$6.A0, U$6.VDD, U1.VDD
- new net GND: D1.A, D2.A, J1.1, J2.6, R6.2, SL2.4, SL3.3, U$1.GND, U$2.GND, U$4.GND, U$5.P$1, U$6.GND, U$7.SNS, U1.A0, U1.A1, U1.GND
- new net N$1: U$1.PTE17, U$2.RXD
- new net N$10: C4.2, R5.1, U$7.VDD
- new net N$11: BAT-.P, C4.1, R6.1, U$7.VSS
- new net N$12: R4.1, U$7.VIN
- new net N$13: D1.C, R7.2, U$7.SCL
- new net N$14: D2.C, R8.2, U$7.SDA
- new net N$15: J2.5, J2.7
- new net N$16: J1.5, J1.7
- new net N$17: J2.2, U$1.PTA14
- new net N$18: J1.3, U$1.PTA15
- new net N$19: BAT+.P, R4.2, R5.2
- new net N$2: U$1.PTE16, U$2.TXD
- new net N$20: J2.3, U$1.PTA16
- new net N$21: J1.4, U$1.PTA17
- new net N$3: U$1.PTE2, U$5.P$6
- new net N$38: U$1.SDA_PTD5
- new net N$39: U$1.AREF
- new net N$4: PAD1.P, U$2.RF_IN
- new net N$40: U$1.VIN
- new net N$41: U$1.5V
- new net N$5: U$1.PTE3, U$5.P$5
- new net N$6: U$1.PTB0, U$5.P$7
- new net N$60: PTE6.P, U$1.PTE6
- new net N$7: U$1.PTB1, U$5.P$8
- new net N$8: U$1.PTA5, U$5.P$3
- new net N$9: U$1.PTA4, U$5.P$4
- new net SCL1: SL3.2, U$1.PTE1, U$4.SCL, U$6.SCL, U1.SCL
- new net SCL2: R7.1, SL2.1, U$1.PTC8, U$5.P$10
- new net SDA1: SL3.1, U$1.PTE0, U$4.SDA, U$6.SDA, U1.SDA
- new net SDA2: R8.1, SL2.3, U$1.PTC9, U$5.P$9
Other:
- note added: "MAX4409 światło"
- note added: "burza"
- note added: "ciśnienie"
- note added: "modół GPS"
- note added: "radio"
- note added: "temperatura"
- note added: "wilgotność"
- note added: "ładowarka ogniwo"
