File: pcb/bord cyfrowy uszko/uszko.brd (EAGLE design)
At the start: 64.8 x 67 mm, 24 parts, among them U1 ADT7410TRZ

Commit message: pcb uszko
Parts:
- removed PTE6: (no value), wirepad:2,54/0,8
- added IC1: REG1117, burr-brown:SOT223
- moved R4 21.7 mm to (59.8, 62.2), turned to 90 degrees
- moved BAT+ 19.6 mm to (62.4, 67.4)
- moved BAT- 19.2 mm to (59.9, 57.8)
- moved R6 19.1 mm to (55.9, 56.0)
- moved C4 15.7 mm to (54.7, 64.0), turned to 0 degrees
- moved D1 15.2 mm to (45.0, 59.6), turned to 180 degrees
- moved R5 14.7 mm to (56.4, 67.4)
- moved R8 12.3 mm to (47.2, 65.8), turned to 180 degrees
- moved D2 10.9 mm to (45.0, 61.9), turned to 180 degrees
- moved R7 5.24 mm to (47.6, 56.9), turned to 180 degrees
- moved U$7 4.02 mm to (53.3, 61.0), turned to 180 degrees
Connections:
- removed net N$60: PTE6.1, U$1.P$48
- net +5V/1: now also IC1.2
- net GND: now also IC1.1
- net N$19: now also IC1.3
Routing:
- net N$9: track 0.00 -> 141.7 mm
- net N$8: track 0.00 -> 126.4 mm
- net SDA2: track 0.00 -> 120.5 mm
- net SCL1: track 12.5 -> 129.9 mm, vias 0 -> 2
- net SCL2: track 0.00 -> 96.2 mm, vias 0 -> 2
- net +5V/1: track 92.2 -> 188.0 mm, vias 2 -> 4
- net SDA1: track 48.8 -> 116.8 mm, vias 2 -> 3
- net N$19: track 0.00 -> 51.5 mm, vias 0 -> 1
- net N$21: track 0.00 -> 33.1 mm
- net N$17: track 0.00 -> 16.3 mm
- net N$11: track 0.00 -> 13.8 mm
- net N$3: track 0.00 -> 12.9 mm
- net N$15: track 0.00 -> 11.2 mm
- net N$5: track 0.00 -> 11.1 mm
- net N$20: track 0.00 -> 9.77 mm
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- added copper zone on layer 16, net GND
Other:
- board size 64.8 x 67 mm -> 68.6 x 70.8 mm

Commit message: bord uszko, piout update
Parts:
- added R1: 1K, resistor:M0805
- added R10, R2, R3, R9: 10K, resistor:M0805
- added T1: (no value), transistor:SOT23-BCE
Connections:
- new net INTER: SL2.2, U$1.P$21
- new net N$22: J1.2, U$1.P$23
- new net N$23: T1.C, U$2.A23
- new net N$24: R1.1, U$1.P$48
- new net N$25: R1.2, T1.B
- new net N$26: J2.1, U$1.P$33
- net +5V/1: now also R10.1, R2.1, R3.1, R9.1, T1.E; no longer U$2.A23
- net SCL1: now also R3.2
- net SCL2: now also R10.2
- net SDA1: now also R2.2
- net SDA2: now also R9.2
Routing:
- net N$22: track 0.00 -> 45.4 mm, vias 0 -> 1
- net INTER: track 0.00 -> 18.1 mm
- net N$23: track 0.00 -> 15.0 mm, vias 0 -> 2
- net +5V/1: track 188.0 -> 201.2 mm
- net N$16: track 0.00 -> 11.2 mm
- net N$26: track 0.00 -> 8.67 mm
- net SCL1: track 129.9 -> 135.3 mm
- net SCL2: track 96.2 -> 100.1 mm
- net SDA1: track 116.8 -> 119.8 mm
- net N$24: track 0.00 -> 2.86 mm
- net SDA2: track 120.5 -> 123.0 mm
- net GND: track 35.0 -> 37.1 mm, vias 8 -> 9
- net N$25: track 0.00 -> 1.89 mm

Commit message: mgr, pcb uszko
Parts:
- moved SL3 19.1 mm to (31.2, 36.8), turned to 270 degrees
- moved SL2 17.8 mm to (30.5, 55.9), turned to 90 degrees
- moved R9 4.02 mm to (34.3, 30.5), turned to 270 degrees
Connections:
- removed net N$2: U$1.P$46, U$2.A20
- new net N$27: U$1.P$44, U$2.A20
- net N$1: now also U$1.P$46; no longer U$1.P$44
Routing:
- net SDA1: track 119.8 -> 138.1 mm, vias 3 -> 4
- net +5V/1: track 201.2 -> 218.4 mm
- net INTER: track 18.1 -> 34.1 mm
- net SDA2: track 123.0 -> 138.4 mm, vias 0 -> 1
- net N$18: track 0.00 -> 14.9 mm
- net N$2: track 13.4 -> 0.00 mm
- net N$27: track 0.00 -> 12.3 mm
- net SCL1: track 135.3 -> 129.0 mm, vias 2 -> 3
- net SCL2: track 100.1 -> 98.7 mm, vias 2 -> 1
- net N$1: track 12.1 -> 12.9 mm, vias 1 -> 0
- net GND: vias 9 -> 10

Commit message: + ADC
Parts:
- removed J1, J2: (no value), con-amp:10X07MTA
- added R11, R12, R13: 1K, resistor:M0805
- added U$3: 2X7PIN, ref-packages:2X7PINCON
Connections:
- new net N$28: R12.2, U$2.A18
- new net N$29: R11.2, U$2.A19
- new net N$30: R13.2, U$2.A17
- net +5V/1: now also U$3.P$13; no longer J1.6
- net GND: now also R11.1, U$3.P$2, U$3.P$8; no longer J1.1, J2.6
- net N$15: now also U$3.P$1, U$3.P$3; no longer J2.5, J2.7
- net N$16: now also U$3.P$12, U$3.P$14; no longer J1.5, J1.7
- net N$17: now also U$3.P$6; no longer J2.2
- net N$18: now also U$3.P$10; no longer J1.3
- net N$20: now also U$3.P$5; no longer J2.3
- net N$21: now also U$3.P$11; no longer J1.4
- net N$22: now also U$3.P$9; no longer J1.2
- net N$23: now also R12.1, R13.1
- net N$26: now also U$3.P$7; no longer J2.1
Routing:
- net N$23: track 15.0 -> 33.3 mm, vias 2 -> 3
- net N$28: track 0.00 -> 4.74 mm
- net N$30: track 0.00 -> 4.63 mm
- net N$29: track 0.00 -> 4.28 mm
- net N$18: track 14.9 -> 11.0 mm
- net N$22: track 45.4 -> 48.1 mm
- net N$15: track 11.2 -> 8.48 mm
- net N$17: track 16.3 -> 13.8 mm, vias 0 -> 2
- net N$21: track 33.1 -> 35.0 mm
- net N$20: track 9.77 -> 7.94 mm
- net +5V/1: track 218.4 -> 220.1 mm
- net N$16: track 11.2 -> 9.53 mm
- net N$26: track 8.67 -> 7.82 mm
