File: pcb/bord wifi uszko/uszko.sch (EAGLE design)
At the start: 7 parts

Commit message: mgr
Other:
- note added: "CC3000 TEXAS WI-FI"
- note added: "TI LAUNCHPAD"
Changed lines of the file:
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@@
 GND
 </text>
-<text x="27.94" y="111.76" size="1.778" layer="92">RFM23</text>
+<text x="27.94" y="109.22" size="5.08" layer="92">RFM23</text>
+<text x="99.314" y="109.728" size="3.302" layer="92">CC3000 TEXAS WI-FI</text>
+<text x="25.4" y="25.4" size="3.556" layer="92">TI LAUNCHPAD</text>
 </plain>
 <instances>
